File: custom-keeb-pcb.kicad_pcb (KiCad board)
At the start: 2 copper layers, 65 x 78.6 mm, 34 parts, among them SW1 SW_Push, SW2 RotaryEncoder_Switch, U1 ATmega32U4-A, Y1 16MHz

Commit message: Finished v2 Design
Rerouted traces, added fill, added decals & text. Ready for printing
Parts:
- added G1: LOGO, Custom_Images:pcbjack, F.Cu at (152.8, 66.4)
- added REF**: MountingHole_2.2mm_M2_Pad, MountingHole:MountingHole_2.2mm_M2_Pad, F.Cu at (177.3, 136.0)
- added REF**: MountingHole_2.2mm_M2_Pad, MountingHole:MountingHole_2.2mm_M2_Pad, F.Cu at (119.3, 136.1)
- moved SW1 37.2 mm to (158.6, 65.0), turned to 0 degrees
- moved R1 21.1 mm to (141.5, 62.9), turned to 0 degrees
- moved R4 16.9 mm to (125.6, 81.3)
- moved C3 16.9 mm to (125.7, 78.1)
- moved C1 14.4 mm to (137.0, 82.5)
- moved C5 14.4 mm to (146.1, 76.7)
- moved C6 14.4 mm to (120.2, 75.3)
- moved C7 14.4 mm to (120.1, 66.4)
- moved C4 14.4 mm to (133.1, 62.5)
- moved U1 14.4 mm to (136.9, 71.6)
- moved Y1 14.4 mm to (120.2, 70.9)
- moved C2 14.2 mm to (146.2, 66.7)
- moved F1 9.90 mm to (166.4, 72.3)
Connections:
- U1 pad 10: COL1 -> ROW1
- U1 pad 11: COL0 -> ROW2
- U1 pad 28: ROW0 -> unconnected-(U1-PB4-Pad28)
- U1 pad 29: ROW1 -> unconnected-(U1-PB5-Pad29)
- U1 pad 30: ROW2 -> unconnected-(U1-PB6-Pad30)
- U1 pad 38: unconnected-(U1-PF5-Pad38) -> COL2
- U1 pad 39: unconnected-(U1-PF4-Pad39) -> COL1
- U1 pad 40: unconnected-(U1-PF1-Pad40) -> COL0
- U1 pad 9: COL2 -> ROW0
Routing:
- net ROW2: track 167.2 -> 118.0 mm, vias 2 -> 0
- net ROW0: track 117.5 -> 76.4 mm, vias 2 -> 0
- net ROW1: track 137.5 -> 98.0 mm, vias 2 -> 0
- net COL2: track 73.9 -> 105.9 mm, vias 3 -> 2
- net PAD1-A: track 34.2 -> 51.4 mm, vias 2 -> 6
- net COL1: track 48.2 -> 64.1 mm, vias 0 -> 2
- net Net-(U1-~{HWB}/PE2): track 18.7 -> 3.20 mm
- net Net-(U1-D+): track 26.2 -> 39.3 mm
- net Net-(U1-D-): track 24.2 -> 36.1 mm
- net RESET: track 43.6 -> 52.5 mm
- net VCC: track 13.6 -> 5.17 mm
- net COL0: track 68.2 -> 76.1 mm, vias 0 -> 2
- net +5V: track 98.4 -> 106.2 mm, vias 7 -> 5
- net PAD1-B: track 47.6 -> 51.8 mm, vias 5 -> 2
- net Net-(D3-A): track 9.56 -> 11.3 mm
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- added copper zone on B.Cu, net GND
Other:
- board size 65 x 78.6 mm -> 64.9 x 78.2 mm
- board text added: "8/1 Macropad v1 Wow!"
- board text added: "JLCJLCJLCJLC"
